File: hw/keynjector/keynjector_mcu.sch (KiCad schematic (older format))
At the start: 21 parts, among them SW1 EVQ-P7L01P, U3 ATSAM4S8BA-ANR

Commit message: added license text to KiCad sheets
Other:
- note added: "Copyright 2014 Jonas Hagmar\n\nThis file is part of keynjector.\n\nkeynjector is free software: you can redistribute it and/or modify\nit under the terms of the GNU General Public License as published by\nthe Free Software Foundation, either version 2 of the License, or\n(at your option) any later version.\n\nkeynjector is distributed in the hope that it will be useful,\nbut WITHOUT ANY WARRANTY;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"
Changed lines of the file:
@@
 Sheet 3 7
 Title ""
-Date "6 nov 2014"
+Date "2 dec 2014"
 Rev ""
 Comp ""
@@
 $EndComp
 Connection ~ 8750 6250
+Text Notes 700  800  0    39   ~ 0
+Copyright 2014 Jonas Hagmar\n\nThis file is part of keynjector.\n\nkeynjector is free software: you can redistribute it and/or modify\nit under the terms of the GNU General Public License as published by\nthe Free Software Foundation, either version 2 of the License, or\n(at your option) any later version.\n\nkeynjector is distributed in the hope that it will be useful,\nbut WITHOUT ANY WARRANTY; without even the implied warranty of\nMERCHANTABILITY or FITNESS FOR A PARTICULAR PURPOSE.  See the\nGNU General Public License for more details.\n\nYou should have received a copy of the GNU General Public License\nalong with keynjector.  If not, see <http://www.gnu.org/licenses/>
 $EndSCHEMATC
