File: hw/zifbrkout/zifbrkout.kicad_pcb (KiCad board)
At the start: 2 copper layers, 33.4 x 39.6 mm, 122 parts, among them J1 501951-4000

Commit message: added copyright notices added COPYING file with GPL v2 license added README file moved font files
Other:
- board text added: "/* * Copyright 2014 Jonas Hagmar * * This file is part of keynjector. * * keynjector is free software: you can redistribute it and/or modify * it under the terms of the GNU General Public License as published by * the Free Software Foundation, either version 2 of the License, or * (at your option) any later version. * * keynjector is distributed in the hope that it will be useful, * but WITHOUT A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"
Changed lines of the file:
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@@
     (area 30.7726 12.8726 65.650001 53.950001)
     (thickness 1.6)
-    (drawings 47)
+    (drawings 48)
     (tracks 314)
     (zones 0)
@@
     )
   )
+  (gr_text "/*\n* Copyright 2014 Jonas Hagmar\n*\n* This file is part of keynjector.\n*\n* keynjector is free software: you can redistribute it and/or modify\n* it under the terms of the GNU General Public License as published by\n* the Free Software Foundation, either version 2 of the License, or\n* (at your option) any later version.\n*\n* keynjector is distributed in the hope that it will be useful,\n* but WITHOUT ANY WARRANTY; without even the implied warranty of\n* MERCHANTABILITY or FITNESS FOR A PARTICULAR PURPOSE.  See the\n* GNU General Public License for more details.\n*\n* You should have received a copy of the GNU General Public License\n* along with keynjector.  If not, see <http://www.gnu.org/licenses/>.\n*/" (at 80.58 22.04) (layer Cmts.User)
+    (effects (font (size 1.5 1.5) (thickness 0.3)) (justify left))
+  )
   (gr_text ":-)" (at 35.1 47.2) (layer B.Mask)
